Commit message: using base_footprint as top frame changing posture of robot in urdf adding Dockerfile

File: pepper_description/urdf/pepper1.0_generated_urdf/pepper.urdf (robot description, URDF)
Before this commit: robot JulietteY20MP, 83 links, 82 joints
Joints:
- joint LElbowRoll: origin xyz=0 0 0 rpy=0 0 0 -> xyz=0 0 0 rpy=0 0 0.79
- joint LShoulderPitch: origin xyz=-0.057 0.14974 0.08682 rpy=0 0 0 -> xyz=-0.057 0.14974 0.08682 rpy=0 1.5 0
- joint LShoulderRoll: origin xyz=0 0 0 rpy=0 0 0 -> xyz=0 0 0 rpy=0 0 -0.79
- joint LWristYaw: origin xyz=0.15 0 0 rpy=0 0 0 -> xyz=0.15 0 0 rpy=-1.6 0 0
- joint RElbowRoll: origin xyz=0 0 0 rpy=0 0 0 -> xyz=0 0 0 rpy=0 0 -0.79
- joint RShoulderPitch: origin xyz=-0.057 -0.14974 0.08682 rpy=0 0 0 -> xyz=-0.057 -0.14974 0.08682 rpy=0 1.5 0
- joint RShoulderRoll: origin xyz=0 0 0 rpy=0 0 0 -> xyz=0 0 0 rpy=0 0 0.79
- joint RWristYaw: origin xyz=0.15 0 0 rpy=0 0 0 -> xyz=0.15 0 0 rpy=1.6 0 0
- joint base_footprint_joint: child base_footprint -> base_link; origin xyz=0 0 -0.334 rpy=0 0 0 -> xyz=0 0 0.82 rpy=0 0 0; parent Tibia -> base_footprint
